File: MicroBrute Noise add-on.brd (EAGLE design)
At the start: 16.1 x 25.5 mm, 20 parts, among them IC1 TL071D, Q1 mmbt3904, Q2 mmbt3904, Q3 mmbt3904

Commit message: touchup
Parts:
- removed FRAME1: FRAME-LETTER, SparkFun-Aesthetics:CREATIVE_COMMONS
Changed lines of the file:
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@@
 <attribute name="PROD_ID" value="CAP-00810" x="14.01" y="20.71" size="1.778" layer="27" rot="R270" display="off"/>
 </element>
-<element name="FRAME1" library="SparkFun-Aesthetics" package="CREATIVE_COMMONS" value="FRAME-LETTER" x="-101.6" y="16.51"/>
 <element name="IC1" library="linear" package="SO08" value="TL071D" x="8.23" y="19.51" rot="R270"/>
 <element name="Q1" library="SparkFun-DiscreteSemi" package="SOT23-3" value="mmbt3904" x="8.59" y="2.38">
