File: MicroBrute Noise add-on.sch (EAGLE design)
At the start: 20 parts, among them IC1 TL071D, Q1 mmbt3904, Q2 mmbt3904, Q3 mmbt3904

Commit message: touchup
Parts:
- removed FRAME1: FRAME-LETTER, SparkFun-Aesthetics:FRAME-LETTER
Changed lines of the file:
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@@
 <setting verticaltext="up"/>
 </settings>
-<grid distance="0.1" unitdist="inch" unit="mil" style="lines" multiple="10" display="no" altdistance="0.01" altunitdist="mm" altunit="mm"/>
+<grid distance="0.1" unitdist="inch" unit="inch" style="lines" multiple="1" display="no" altdistance="0.01" altunitdist="inch" altunit="inch"/>
 <layers>
 <layer number="1" name="Top" color="4" fill="1" visible="no" active="no"/>
@@
 <schematic xreflabel="%F%N/%S.%C%R" xrefpart="/%S.%C%R">
 <attributes>
+<attribute name="CNAME" value="Microbrute Addon"/>
+<attribute name="CREVISION" value="1"/>
+<attribute name="DESIGNER" value="Gilberte / Mads Kjeldgaard"/>
 </attributes>
 <variantdefs>
@@
 </classes>
 <parts>
-<part name="FRAME1" library="SparkFun-Aesthetics" deviceset="FRAME-LETTER" device=""/>
 <part name="C1" library="SparkFun-Passives" deviceset="CAP_POL" device="C" value="10uf"/>
 <part name="Q1" library="SparkFun-DiscreteSemi" deviceset="TRANSISTOR_NPN" device="SOT23-3" value="mmbt3904"/>
@@
 <part name="SUPPLY4" library="supply2" deviceset="VEE" device=""/>
 <part name="GND2" library="SparkFun" deviceset="GND" device=""/>
+<part name="FRAME1" library="SparkFun-Aesthetics" deviceset="FRAME-A4L" device=""/>
 </parts>
 <sheets>
@@
 </plain>
 <instances>
-<instance part="FRAME1" gate="G$1" x="0" y="0"/>
-<instance part="FRAME1" gate="V" x="147.32" y="0"/>
 <instance part="C1" gate="G$1" x="17.78" y="78.74"/>
 <instance part="Q1" gate="G$1" x="53.34" y="68.58"/>
@@
 <instance part="SUPPLY4" gate="G$1" x="190.5" y="147.32" rot="R90"/>
 <instance part="GND2" gate="1" x="187.96" y="132.08" rot="R270"/>
+<instance part="FRAME1" gate="G$1" x="4.064" y="3.556"/>
 </instances>
 <busses>
