File: White Noise Addon/MicroBrute Noise add-on.brd (EAGLE design)
At the start: 16.1 x 25.5 mm, 21 parts, among them IC1 TL071D, Q1 mmbt3904, Q2 mmbt3904, Q3 mmbt3904

Commit message: cleanup
Parts:
- added GND5: TEST-POINT3X5, SparkFun-Passives:PAD.03X.05
Connections:
- net GND: now also GND5.P$1
Routing:
- net GND: track 49.4 -> 60.2 mm
Changed lines of the file:
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@@
 Thomas Henry, Walter
 G. Jung, Olivier Gillet. </text>
+<circle x="2.1" y="2.4" radius="1.334165625" width="0.1" layer="22"/>
+<text x="2.96" y="3.735" size="0.6096" layer="26" rot="MR0">GND</text>
 </plain>
 <attributes>
@@
 <element name="D2" library="diode" package="SOD523" value="PMEG2010AEB" x="8.2" y="24" rot="MR0"/>
 <element name="D1" library="diode" package="SOD523" value="PMEG2010AEB" x="4.8" y="24.1" rot="MR0"/>
+<element name="GND5" library="SparkFun-Passives" package="PAD.03X.05" value="TEST-POINT3X5" x="2.1" y="2.5" rot="MR0"/>
 </elements>
 <signals>
@@
 <wire x1="4.4704" y1="7.3152" x2="4.4704" y2="5.08" width="0.2032" layer="16"/>
 <wire x1="6.7056" y1="9.5504" x2="4.4704" y2="7.3152" width="0.2032" layer="16"/>
-<wire x1="6.7056" y1="10.7696" x2="6.7056" y2="9.5504" width="0.2032" layer="16"/>
+<wire x1="6.7056" y1="10.5664" x2="6.7056" y2="9.5504" width="0.2032" layer="16"/>
 <wire x1="6.7056" y1="15.0368" x2="6.7056" y2="10.7696" width="0.2032" layer="1"/>
 <wire x1="7.7216" y1="16.0528" x2="6.7056" y2="15.0368" width="0.2032" layer="1"/>
@@
 <wire x1="11.176" y1="6.096" x2="11.29" y2="5.9" width="0.2032" layer="16"/>
 <via x="6.7056" y="10.7696" extent="1-16" drill="0.508"/>
+<contactref element="GND5" pad="P$1"/>
+<wire x1="2.2352" y1="7.5184" x2="2.2352" y2="2.6416" width="0.2032" layer="16"/>
+<wire x1="5.2832" y1="10.5664" x2="2.2352" y2="7.5184" width="0.2032" layer="16"/>
+<wire x1="6.7056" y1="10.5664" x2="5.2832" y2="10.5664" width="0.2032" layer="16"/>
+<wire x1="2.2352" y1="2.6416" x2="2.1" y2="2.5" width="0.2032" layer="16"/>
+<wire x1="6.7056" y1="10.5664" x2="6.7056" y2="10.7696" width="0.2032" layer="16"/>
 </signal>
 <signal name="VEE">
@@
 <vertex x="0" y="25.5"/>
 </polygon>
+<wire x1="5.2832" y1="4.8768" x2="5.406396875" y2="4.999996875" width="0.2032" layer="16"/>
+<wire x1="6.5024" y1="8.5344" x2="6.45520625" y2="8.581590625" width="0.2032" layer="16"/>
 </signal>
 <signal name="N$8">
